Commit message: chore: Update simulations

File: control/InverseKinematics/urdfs/back_up.urdf (robot description, URDF)
Before this commit: robot complex_robot, 6 links, 5 joints
Links:
- removed link base_link
- removed link link5
- added link base; visual box size=0.2 0.2 0.1
- link link1: geometry visual cylinder length=0.03 radius=0.02
- link link2: geometry visual cylinder length=0.25 radius=0.02
- link link3: geometry visual cylinder length=0.28 radius=0.02
- link link4: geometry visual cylinder length=0.28 radius=0.02
Joints:
- joint joint1: origin xyz=0 0 0.05 rpy=0 0 0 -> xyz=0 0 0.1 rpy=0 0 0; parent base_link -> base
- joint joint2: axis 0 0 1 -> 0 1 0; origin xyz=0 0 0.4 rpy=0 0 0 -> xyz=0 0 0.03 rpy=0 0 0
- joint joint3: axis 0 0 1 -> 0 1 0; origin xyz=0 0 0.3 rpy=0 0 0 -> xyz=0 0 0.25 rpy=0 0 0
- joint joint4: axis 0 0 1 -> 0 1 0; origin xyz=0 0 0.25 rpy=0 0 0 -> xyz=0 0 0.28 rpy=0 0 0
- joint joint5: axis 0 0 1 -> 0 1 0; child link5 -> link4; origin xyz=0 0 0.2 rpy=0 0 0 -> xyz=0 0 0.28 rpy=0 0 0

File: control/InverseKinematics/urdfs/s.urdf (robot description, URDF)
Before this commit: robot complex_robot, 6 links, 5 joints
Links:
- link link1: geometry visual cylinder length=0.03 radius=0.02
- link link2: geometry visual cylinder length=0.25 radius=0.02
- link link3: geometry visual cylinder length=0.28 radius=0.02
- link link4: geometry visual cylinder length=0.28 radius=0.02
Joints:
- joint joint2: origin xyz=0 0 0.4 rpy=0 0 0 -> xyz=0 0 0.03 rpy=0 0 0
- joint joint3: origin xyz=0 0 0.3 rpy=0 0 0 -> xyz=0 0 0.25 rpy=0 0 0
- joint joint4: origin xyz=0 0 0.25 rpy=0 0 0 -> xyz=0 0 0.28 rpy=0 0 0
- joint joint5: origin xyz=0 0 0.2 rpy=0 0 0 -> xyz=0 0 0.28 rpy=0 0 0

Commit message: Refactor inverse kinematics code for improved readability and maintainability

File: control/InverseKinematics/urdfs/back_up.urdf (robot description, URDF)
Before this commit: robot optimized_complex_robot, 5 links, 5 joints
Links:
- added link link5; visual cylinder length=0.15 radius=0.02
Joints:
- joint joint1: origin xyz=0 0 0.1 rpy=0 0 0 -> xyz=0 0 0.05 rpy=0 0 0
- joint joint5: child link4 -> link5

File: control/InverseKinematics/urdfs/s.urdf (robot description, URDF)
Before this commit: robot optimized_complex_robot, 6 links, 5 joints
Links:
- link link5: geometry visual box size=0.05 0.05 0.02
