Commit message: Refactor FK calculation

File: control/InverseKinematics/urdfs/s.urdf (robot description, URDF)
Before this commit: robot optimized_complex_robot, 6 links, 5 joints
Links:
- link base: geometry visual box size=0.07 0.07 0.1
- link link2: geometry visual cylinder length=0.3 radius=0.02
- link link3: geometry visual cylinder length=0.3 radius=0.02
- link link4: geometry visual cylinder length=0.3 radius=0.02
- link link5: geometry visual cylinder length=0.1 radius=0.02
Joints:
- joint joint3: origin xyz=0 0 0.25 rpy=0 0 0 -> xyz=0 0 0.3 rpy=0 0 0
- joint joint4: origin xyz=0 0 0.28 rpy=0 0 0 -> xyz=0 0 0.3 rpy=0 0 0
- joint joint5: origin xyz=0 0 0.28 rpy=0 0 0 -> xyz=0 0 0.3 rpy=0 0 0

Commit message: Refactor FK calculation code

File: control/InverseKinematics/urdfs/s.urdf (robot description, URDF)
Before this commit: robot optimized_complex_robot, 6 links, 5 joints
Joints:
- joint joint5: axis 0 1 0 -> 0 0 1

Commit message: Refactor FK calculation code

File: control/InverseKinematics/urdfs/s.urdf (robot description, URDF)
Before this commit: robot optimized_complex_robot, 6 links, 5 joints
Links:
- link link4: geometry visual cylinder length=0 radius=0.02
Joints:
- joint joint5: origin xyz=0 0 0.3 rpy=0 0 0 -> xyz=0 0 0 rpy=0 0 0

Commit message: Refactor workspace generation code and update link lengths in URDF file

File: control/InverseKinematics/urdfs/s.urdf (robot description, URDF)
Before this commit: robot optimized_complex_robot, 6 links, 5 joints
Links:
- link base: geometry visual box size=0.07 0.07 0.07
- link link2: geometry visual cylinder length=0.5 radius=0.02
- link link3: geometry visual cylinder length=0.5 radius=0.02
Joints:
- joint joint1: origin xyz=0 0 0.05 rpy=0 0 0 -> xyz=0 0 0.03 rpy=0 0 0
- joint joint3: origin xyz=0 0 0.3 rpy=0 0 0 -> xyz=0 0 0.5 rpy=0 0 0
- joint joint4: origin xyz=0 0 0.3 rpy=0 0 0 -> xyz=0 0 0.5 rpy=0 0 0
