Commit message: Refactor modeling section

File: Modeling/InverseKinematics/urdfs/s.urdf (robot description, URDF)
Before this commit: robot optimized_complex_robot, 6 links, 5 joints
Links:
- link base: geometry visual box size=0.07 0.07 0.1
Joints:
- joint joint1: origin xyz=0 0 0.03 rpy=0 0 0 -> xyz=0 0 0.1 rpy=0 0 0
